File: hardware/esp32-e220.kicad_pcb (KiCad board)
At the start: 2 copper layers, 145 x 90 mm, 33 parts, among them J1 SSW-115-02-G-S DEVKIT LEFT, J2 SSW-115-02-G-S DEVKIT RIGHT, J3 E220-400T22D / E220-900T22D S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, J4 B2B-XH-A, J5 SSW-104-02-G-S, Q1 DMP3130LQ-7, U1 TPS62133RGT, U3 SN74AHCT1G125DBVR

Commit message: next commit
Parts:
- moved D3 13.3 mm to (41.9, 70.5), turned to 180 degrees
- moved C2 1.30 mm to (75.4, 73.9), turned to -90 degrees
- moved C1 1.04 mm to (75.3, 70.5), turned to -90 degrees
Connections:
- net 5V_SYS renamed /5V_SYS
- net BAT_FUSED renamed /BAT_FUSED
- net BAT_PLUS renamed /BAT_PLUS
- net BUCK_IN renamed /BUCK_IN
- net BUCK_SW renamed /BUCK_SW
- net DEVKIT_3V3 renamed /DEVKIT_3V3
- net E220_AUX renamed /E220_AUX
- net E220_M0 renamed /E220_M0
- net E220_M1 renamed /E220_M1
- net E220_RXD renamed /E220_RXD
- net E220_TXD renamed /E220_TXD
- net GND renamed /GND
- net OLED_SCL renamed /OLED_SCL
- net OLED_SDA renamed /OLED_SDA
- net Q1_GATE renamed /Q1_GATE
- net SS_TR renamed /SS_TR
- net WS2812_DATA_3V3 renamed /WS2812_DATA_3V3
- net WS2812_DIN renamed /WS2812_DIN
Other:
- board text added: "ACTUAL PAD-SIDE CHECK: PVIN→C1 2.58 mm; AVIN→C2 2.20 mm; C1/C2 GND→EP/PGND 3.34/2.92 mm; SW→L1 2.63 mm"
- board text removed: "ACTUAL PAD-SIDE CHECK: PVIN→C1 2.12 mm; AVIN→C2 1.32 mm; SW→L1 2.63 mm; L1→COUT 1.43 mm"
