File: hardware/esp32-e220.kicad_pcb (KiCad board)
At the start: 2 copper layers, 145 x 90 mm, 40 parts, among them J1 SSW-115-02-G-S DEVKIT LEFT, J2 SSW-115-02-G-S DEVKIT RIGHT, J3 E220-400T22D / E220-900T22D S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, J4 B2B-XH-A, J5 SSW-104-02-G-S, J6 BUTTONS 1x6 2.54mm DNP, J8 B2B-XH-A, J9 J_RGB / RGB OUT 1x3 2.54mm DNP, Q1 DMP3130LQ-7, U1 TPS62133RGT, U3 SN74AHCT1G125DBVR, U4 TLV1117LV33DCYR

Commit message: Audit and correct production footprints
Parts:
- JP1: footprint Connector_PinHeader_2.54mm:PinHeader_1x02_P2.54mm_Vertical -> Carrier:Samtec_TSW-102-07-G-S_1x02_P2.54mm_THT
- U4: footprint Package_TO_SOT_SMD:SOT-223-3_TabPin2 -> Carrier:TI_TLV1117LV33DCYR_DCY_SOT223
- moved F1 0.75 mm to (44.2, 76.0)
Routing:
- net /WS2812_DATA_5V: track 12.8 -> 12.2 mm
- net /WS2812_DATA_3V3: track 108.8 -> 108.2 mm
- net /BAT_PLUS: track 22.8 -> 22.3 mm

Commit message: Correct D3 and Murata manufacturer land patterns
Parts:
- C3: footprint Murata_GRM21_2012Metric -> Murata_GRM21BR61A226ME44_2012Metric
- C5: footprint Murata_GRM188_1608Metric -> Murata_GRM188R61A106MAAL_1608Metric
