File: hardware/esp32-e220.kicad_sch (KiCad schematic)
At the start: 21 parts, among them J1 DEVKIT_LEFT (USB-C toward ant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, J2 DEVKIT_RIGHT (USB-C toward an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, J3 E220-900T22D, J4 USB4105-GF-A, Q1 MMBT3904LT1G, U1 TUSB320LAIRWBR, U2 TPS259630DDAR

Commit message: next commit
Parts:
- removed J3: E220-900T22D, symbol Project:E220_900T22D
- added J3: E220-T22D SOCKET — FIT 400T22D OR 900T22D, symbol Project:E220_T22D_400_900
- added R8: 10k 1% M0 reset pull-down, symbol Project:R
- added R9: 10k 1% M1 reset pull-down, symbol Project:R
- C5: value 10uF 10V X5R -> GRM188R61A106MAAL 10uF 10V X5R
- C6: value 100nF 16V X7R -> GRM188R71C104KA01D 100nF 16V X7R
Connections:
- net 5V_SYS: now also J3.6 (VCC)
- net E220_AUX: now also J3.5 (AUX)
- net E220_M0: now also J3.1 (M0), R8.1
- net E220_M1: now also J3.2 (M1), R9.1
- net E220_RXD: now also J3.3 (RXD)
- net E220_TXD: now also J3.4 (TXD)
- net GND: now also J3.7 (GND), R8.2, R9.2
- net OLED_SDA: now reaches J2.11 (GPIO21)
- net OLED_SCL: now reaches J2.14 (GPIO22)
- no-connect marks 22 -> 20
Other:
- note added: "E220 M0/M1 use 10k pull-downs to GND (PROJECT DESIGN CHOICE): reset mode M1/M0=00. AUX is input-only, no pull-down."
- note added: "J3 is universal E220-T22D interface: fit one E220-400T22D OR E220-900T22D. No socket/footprint is selected."
- note added: "OLED: GPIO21/SDA and GPIO22/SCL are signal-only reservations; OLED VCC and I2C pull-ups are NC/DNP in Rev A."
- note added: "Pin-level Type-C and eFuse support components are documented with official PNs and values. Footprints intentionally unassigned at schematic stage."
- note added: "Stage 5 — main board only. DevKit USB-C programming and main-board USB-C power are mutually exclusive (approved Rev A policy)."
- note removed: "E220: firmware drives M0/M1; no unverified external pull resistor. AUX is input-only, no pull-down."
- note removed: "Pin-level Type-C and eFuse support components are documented with their official PNs and values. Footprints intentionally unassigned at schematic stage."
- note removed: "Stage 4 — main board only. DevKit USB-C programming and main-board USB-C power are mutually exclusive (approved Rev A policy)."
- title: ESP32 E220 LoRa Receiver — Stage 4 -> ESP32 E220 LoRa Receiver — Stage 5 modular carrier

Commit message: next commit
Parts:
- removed D1: MMSD4148T1G, symbol Project:D
- removed J4: USB4105-GF-A, symbol Project:USB_C_POWER
- removed Q1: MMBT3904LT1G, symbol Project:MMBT3904LT1G
- removed R3: 47k 0.1%, symbol Project:R
- removed R4: 330k 0.1%, symbol Project:R
- removed R5: 909R 0.1%, symbol Project:R
- removed R6: 365k 0.1%, symbol Project:R
- removed R7: 100k 0.1%, symbol Project:R
- removed U1: TUSB320LAIRWBR, symbol Project:TUSB320LAIRWBR
- removed U2: TPS259630DDAR, symbol Project:TPS259630DDAR
- added C7: GRM188R71C104KA01D 100nF 16V X7R, symbol Project:C
- added D2: WS2812B-V5, symbol Project:WS2812B_V5
- added D3: SMBJ10CA (bidirectional TVS), symbol Project:TVS
- added F1: 1812L200/16 (2A hold PPTC), symbol Project:F
- added J4: PROTECTED 2S LI-ION INPUT ONLY 6...8.4V, symbol Project:Battery_2S_Protected_Input
- added J5: OLED 0.96 SSD1306 128x64 I2C — FEMALE 1x4 SOCKET, symbol Project:OLED_SSD1306_I2C_1x4
- added L1: XFL4020-222MEB 2.2uH, symbol Project:L
- added Q1: DMP3130LQ-7 (reverse-polarity), symbol Project:DMP3130LQ_7
- added R10: DNP 4.7k 1% OLED SDA pull-up to 3V3, symbol Project:R
- added R11: DNP 4.7k 1% OLED SCL pull-up to 3V3, symbol Project:R
- added TP1: BAT_PLUS, symbol Project:TestPoint
- added TP10: E220_TXD, symbol Project:TestPoint
- added TP2: GND, symbol Project:TestPoint
- added TP3: BUCK_IN, symbol Project:TestPoint
- added TP4: 5V_SYS, symbol Project:TestPoint
- added TP5: E220_VCC, symbol Project:TestPoint
- added TP6: E220_M0, symbol Project:TestPoint
- added TP7: E220_M1, symbol Project:TestPoint
- added TP8: E220_AUX, symbol Project:TestPoint
- added TP9: E220_RXD, symbol Project:TestPoint
- added U1: TPS62133RGT (5V / 3A BUCK), symbol Project:TPS62133RGT
- added U3: SN74AHCT1G125DBVR, symbol Project:SN74AHCT1G125DBVR
- C1: value 1uF 10V X7R -> GRM21BR61E106KA73 10uF 25V X5R (BUCK IN)
- C2: value 100nF 16V X7R -> GRM188R71C104KA01D 100nF 16V X7R (AVIN)
- C3: value 1uF 10V X7R -> GRM21BR61A226ME44 22uF 10V X5R (BUCK OUT)
- C4: value 3.3nF 50V C0G -> GRM1885C1H332JA01D 3.3nF 50V C0G (SS/TR)
- R1: value 900k 1% -> 100k 1% (Q1 gate pull-down)
- R2: value 47k 0.1% -> 1M 1% (Q1 gate-source)
Connections:
- net VBUS_DET is gone; now on net GND: R1.2
- net 5V_SYS: now also C7.1, D2.1 (VDD), L1.2, TP4.1, TP5.1, U1.14 (VOS), U1.7 (FSW), U3.5 (VCC)
- net E220_AUX: now also TP8.1
- net E220_M0: now also TP6.1
- net E220_M1: now also TP7.1
- net E220_RXD: now also TP9.1
- net E220_TXD: now also TP10.1
- net GND: now also C7.2, D2.3 (VSS), D3.2 (K), J4.2 (BAT-), J5.1 (GND), TP2.1, U1.15 (PGND), U1.16 (PGND), U1.5 (FB), U1.6 (AGND), U1.8 (DEF), U1.EP (EXPOSED THERMAL PAD), U3.1 (OE), U3.3 (GND)
- net OLED_SCL: now also J5.3 (SCL), R11.1
- net OLED_SDA: now also J5.4 (SDA), R10.1
- net DEVKIT_3V3: now reaches J2.1 (3V3)
- net DEVKIT_3V3: now also J5.2 (VCC / 3V3), R10.2, R11.2
- net WS2812_DATA_3V3: now reaches J2.5 (GPIO4)
- net WS2812_DATA_3V3: now also U3.2 (A)
- net DVDT renamed SS_TR
- net SS_TR: now also U1.9 (SS/TR)
- net OUT1 renamed Q1_GATE
- net Q1_GATE: now also R1.1, Q1.1 (G)
- net TUSB_VDD renamed BUCK_IN
- net BUCK_IN: now also C1.1, Q1.2 (S), TP3.1, U1.10 (AVIN), U1.11 (PVIN), U1.12 (PVIN), U1.13 (EN)
- removed net VBUS_PRE: C1.1, R1.1
- new net BAT_FUSED: D3.1 (A), F1.2, Q1.3 (D)
- new net BAT_PLUS: F1.1, J4.1 (BAT+), TP1.1
- new net BUCK_SW: L1.1, U1.1 (SW), U1.2 (SW), U1.3 (SW)
- new net WS2812_DIN: D2.4 (DIN), U3.4 (Y)
- no-connect marks 20 -> 21
Other:
- note added: "BAT+ -> F1 1812L200/16 -> BAT_FUSED -> Q1 DMP3130LQ-7 reverse-polarity MOSFET -> BUCK_IN -> U1 TPS62133RGT -> 5V_SYS."
- note added: "D3 SMBJ10CA is a bidirectional input transient clamp at BAT_FUSED. No on-board charger/BMS is duplicated; no main-board switch is fitted in Rev.1."
- note added: "GPIO4 -> SN74AHCT1G125DBVR (OE=GND, 5V) -> WS2812B-V5 DIN. No PCB footprint/layout work is included."
- note added: "J3 is universal E220-T22D: fit one E220-400T22D OR E220-900T22D. M0/M1 10k pulldowns. J5 is removable SSD1306 0.96 I2C, 1 GND/2 3V3/3 SCL/4 SDA."
- note added: "OLED VCC is DEVKIT_3V3 only. R10/R11 optional DNP 4.7k pull-ups to 3V3; fit only after checking module pull-ups. No 5V OLED power or pull-up."
- note added: "Rev.1 active input: externally protected 2S 18650 pack + external BMS only. J4 is BAT+/BAT- 6.0...8.4V; no midpoint, charger or USB-C input."
- note added: "Rev.1 policy: disconnect battery or turn its external BMS output off before connecting the removable DevKit USB-C to a computer for programming."
- note added: "TP1 BAT_PLUS, TP2 GND, TP3 BUCK_IN, TP4 5V_SYS, TP5 E220_VCC(5V_SYS), TP6 M0, TP7 M1, TP8 AUX, TP9 RXD, TP10 TXD."
- note added: "TPS62133: PVIN/AVIN/EN=BUCK_IN, SW1-3 -> L1 2.2uH -> 5V_SYS, VOS/FSW=5V_SYS, FB/DEF/grounds/EP=GND, SS/TR=C4 to GND; PG NC."
- note removed: "E220 M0/M1 use 10k pull-downs to GND (PROJECT DESIGN CHOICE): reset mode M1/M0=00. AUX is input-only, no pull-down."
- note removed: "J3 is universal E220-T22D interface: fit one E220-400T22D OR E220-900T22D. No socket/footprint is selected."
- note removed: "No bare ESP32, 3V3 buck, EN/BOOT or programming circuit on this PCB. J1/J2 are the verified removable DevKit sockets."
- note removed: "OLED: GPIO21/SDA and GPIO22/SCL are signal-only reservations; OLED VCC and I2C pull-ups are NC/DNP in Rev A."
- note removed: "Pin-level Type-C and eFuse support components are documented with official PNs and values. Footprints intentionally unassigned at schematic stage."
- note removed: "Stage 5 — main board only. DevKit USB-C programming and main-board USB-C power are mutually exclusive (approved Rev A policy)."
- note removed: "TUSB320 UFP/GPIO: PORT=GND, ADDR=NC, EN_N=GND. OUT1/Q1 gates TPS259630: Default/detach OFF; Medium/High ON."
- title: ESP32 E220 LoRa Receiver — Stage 5 modular carrier -> ESP32 E220 LoRa Receiver — Rev.1 protected 2S battery carrier

Commit message: next commit
Connections:
- net GND is gone; now on net 5V_SYS: C1.2, C2.2, C3.2, C4.2, C5.2, C6.2, C7.2, D2.3 (VSS), D3.2 (K), J1.2 (GND), J2.2 (GND), J3.7 (GND), J4.2 (BAT-), J5.1 (GND), R1.2, R8.2, R9.2, TP2.1, U1.15 (PGND), U1.16 (PGND), U1.5 (FB), U1.6 (AGND), U1.8 (DEF), U1.EP (EXPOSED THERMAL PAD), U3.1 (OE), U3.3 (GND)
- no-connect marks 21 -> 20
Other:
- note added: "0.96" SSD1306 | 128x64 | I2C | USER INSTALLED"
- note added: "30 PIN / 2x15 | USB-C + CH340C ON MODULE"
- note added: "A. BATTERY INPUT / PROTECTION"
- note added: "B. 2S -> 5V BUCK"
- note added: "BAT+ -> F1 -> BAT_FUSED -> Q1 -> BUCK_IN"
- note added: "C. REMOVABLE ESP32 DEVKIT"
- note added: "D. E220-T22D UNIVERSAL SOCKET"
- note added: "D3 TVS"
- note added: "E. REMOVABLE OLED"
- note added: "E220-400T22D / E220-900T22D — user-installed module"
- note added: "ESP32 DEVKIT, E220 AND OLED ARE USER-INSTALLED MODULES."
- note added: "F. WS2812 STATUS LED"
- note added: "GND"
- note added: "GPIO4 -> AHCT buffer -> DIN"
- note added: "Inter-block links use net labels. Local wires show the active power, bypass and interface support networks."
- note added: "J5: 1 GND | 2 DEVKIT_3V3 | 3 GPIO22/SCL | 4 GPIO21/SDA | R10/R11 4.7k DNP"
- note added: "LEFT HEADER: J1 RIGHT HEADER: J2"
- note added: "POWER INPUT: EXTERNALLY PROTECTED 2S LI-ION | 6.0 ... 8.4 V | NO CHARGER ON CARRIER PCB"
- note added: "U1 TPS62133RGT: C1 10uF input | C2 100nF AVIN | C4 3.3nF SS | L1 2.2uH | C3 22uF output"
- note added: "USED: VIN, 3V3, GND | GPIO17/TX2, GPIO16/RX2, GPIO25/26/27, GPIO21/22, GPIO4"
- note added: "WARNING: TURN OFF / DISCONNECT BATTERY POWER BEFORE CONNECTING ESP32 DEVKIT USB-C TO A COMPUTER."
- note added: "|"
- note removed: "BAT+ -> F1 1812L200/16 -> BAT_FUSED -> Q1 DMP3130LQ-7 reverse-polarity MOSFET -> BUCK_IN -> U1 TPS62133RGT -> 5V_SYS."
- note removed: "D3 SMBJ10CA is a bidirectional input transient clamp at BAT_FUSED. No on-board charger/BMS is duplicated; no main-board switch is fitted in Rev.1."
- note removed: "GPIO4 -> SN74AHCT1G125DBVR (OE=GND, 5V) -> WS2812B-V5 DIN. No PCB footprint/layout work is included."
- note removed: "J3 is universal E220-T22D: fit one E220-400T22D OR E220-900T22D. M0/M1 10k pulldowns. J5 is removable SSD1306 0.96 I2C, 1 GND/2 3V3/3 SCL/4 SDA."
- note removed: "OLED VCC is DEVKIT_3V3 only. R10/R11 optional DNP 4.7k pull-ups to 3V3; fit only after checking module pull-ups. No 5V OLED power or pull-up."
- note removed: "Rev.1 active input: externally protected 2S 18650 pack + external BMS only. J4 is BAT+/BAT- 6.0...8.4V; no midpoint, charger or USB-C input."
- note removed: "Rev.1 policy: disconnect battery or turn its external BMS output off before connecting the removable DevKit USB-C to a computer for programming."
- note removed: "TP1 BAT_PLUS, TP2 GND, TP3 BUCK_IN, TP4 5V_SYS, TP5 E220_VCC(5V_SYS), TP6 M0, TP7 M1, TP8 AUX, TP9 RXD, TP10 TXD."
- note removed: "TPS62133: PVIN/AVIN/EN=BUCK_IN, SW1-3 -> L1 2.2uH -> 5V_SYS, VOS/FSW=5V_SYS, FB/DEF/grounds/EP=GND, SS/TR=C4 to GND; PG NC."

Commit message: next commit
Parts:
- C1: value GRM21BR61E106KA73 10uF 25V X5R (BUCK IN) -> GRM21BR61E106KA73; footprint (none) -> Murata_GRM21_2012Metric
- C2: value GRM188R71C104KA01D 100nF 16V X7R (AVIN) -> GRM188R71C104KA01D; footprint (none) -> Murata_GRM188_1608Metric
- C3: value GRM21BR61A226ME44 22uF 10V X5R (BUCK OUT) -> GRM21BR61A226ME44; footprint (none) -> Murata_GRM21_2012Metric
- C4: value GRM1885C1H332JA01D 3.3nF 50V C0G (SS/TR) -> GRM1885C1H332JA01D; footprint (none) -> Murata_GRM188_1608Metric
- C5: value GRM188R61A106MAAL 10uF 10V X5R -> GRM188R61A106MAAL; footprint (none) -> Murata_GRM188_1608Metric
- C6, C7: value GRM188R71C104KA01D 100nF 16V X7R -> GRM188R71C104KA01D; footprint (none) -> Murata_GRM188_1608Metric
- D2: footprint (none) -> WorldSemi_WS2812B-V5_PLACEMENT_CANDIDATE_NOT_RELEASED
- D3: value SMBJ10CA (bidirectional TVS) -> SMBJ10CA; footprint (none) -> Littelfuse_SMBJ10CA_DO214AA
- F1: value 1812L200/16 (2A hold PPTC) -> 1812L200/16; footprint (none) -> Littelfuse_1812L200_16_4532Metric
- J1: value DEVKIT_LEFT (USB-C toward antenna) -> SSW-115-02-G-S DEVKIT LEFT; footprint (none) -> Samtec_SSW_1x15_P2.54mm_THT
- J2: value DEVKIT_RIGHT (USB-C toward antenna) -> SSW-115-02-G-S DEVKIT RIGHT; footprint (none) -> Samtec_SSW_1x15_P2.54mm_THT
- J3: value E220-T22D SOCKET — FIT 400T22D OR 900T22D -> E220-400T22D / E220-900T22D SOCKET; footprint (none) -> E220_T22D_Socket_400_900
- J4: value PROTECTED 2S LI-ION INPUT ONLY 6...8.4V -> B2B-XH-A; footprint (none) -> JST_B2B-XH-A_1x02_P2.50mm_THT
- J5: value OLED 0.96 SSD1306 128x64 I2C — FEMALE 1x4 SOCKET -> SSW-104-02-G-S; footprint (none) -> Samtec_SSW_1x04_P2.54mm_THT
- L1: value XFL4020-222MEB 2.2uH -> XFL4020-222MEB; footprint (none) -> Coilcraft_XFL4020-222MEB
- Q1: value DMP3130LQ-7 (reverse-polarity) -> DMP3130LQ-7; footprint (none) -> Diodes_DMP3130LQ-7_SOT23
- R1: value 100k 1% (Q1 gate pull-down) -> 100k 1%; footprint (none) -> Resistor_0603_1608Metric
- R2: value 1M 1% (Q1 gate-source) -> 1M 1%; footprint (none) -> Resistor_0603_1608Metric
- R8: value 10k 1% M0 reset pull-down -> 10k 1%; footprint (none) -> Resistor_0603_1608Metric
- R9: value 10k 1% M1 reset pull-down -> 10k 1%; footprint (none) -> Resistor_0603_1608Metric
- TP1, TP10, TP2, TP3, TP4, TP6, TP7, TP8, TP9: footprint (none) -> TestPoint_THT_1p0mm_PROTOTYPE
- TP5: value E220_VCC -> 5V_SYS; footprint (none) -> TestPoint_THT_1p0mm_PROTOTYPE
- U1: value TPS62133RGT (5V / 3A BUCK) -> TPS62133RGT; footprint (none) -> TI_TPS62133RGT_RGT0016C
- U3: footprint (none) -> TI_SN74AHCT1G125DBVR_SOT23-5

Commit message: next commit
Parts:
- removed D2: WS2812B-V5, WorldSemi_WS2812B-V5_PLACEMENT_CANDIDATE_NOT_RELEASED, symbol Project:WS2812B_V5
- removed TP10: E220_TXD, TestPoint_THT_1p0mm_PROTOTYPE, symbol Project:TestPoint
- removed TP6: E220_M0, TestPoint_THT_1p0mm_PROTOTYPE, symbol Project:TestPoint
- removed TP7: E220_M1, TestPoint_THT_1p0mm_PROTOTYPE, symbol Project:TestPoint
- removed TP8: E220_AUX, TestPoint_THT_1p0mm_PROTOTYPE, symbol Project:TestPoint
- removed TP9: E220_RXD, TestPoint_THT_1p0mm_PROTOTYPE, symbol Project:TestPoint
- added C10, C9: GRM21BR61E106KA73, Carrier:Murata_GRM21_2012Metric, symbol Project:C
- added C8: GRM188R71C104KA01D, Carrier:Murata_GRM188_1608Metric, symbol Project:C
- added J6: BUTTONS 1x6 2.54mm DNP, Carrier:PinHeader_1x06_P2.54mm_Vertical, symbol Project:BUTTONS_1x6
- added J8: B2B-XH-A, JST_B2B-XH-A_1x02_P2.50mm_THT, symbol Project:POWER_SW_1x2
- added J9: J_RGB / RGB OUT 1x3 2.54mm DNP, Carrier:PinHeader_1x03_P2.54mm_Vertical, symbol Project:RGB_OUT_1x3
- added JP1: TSW-102-07-G-S + SNT-100-BK-G, Connector_PinHeader_2.54mm:PinHeader_1x02_P2.54mm_Vertical, symbol Project:DEVKIT_PWR_1x2
- added R3: RC0603FR-0710KL, Carrier:Resistor_0603_1608Metric, symbol Project:R
- added R4: RC0603FR-073K3L, Carrier:Resistor_0603_1608Metric, symbol Project:R
- added U4: TLV1117LV33DCYR, Package_TO_SOT_SMD:SOT-223-3_TabPin2, symbol Project:TLV1117LV33DCY
- R10: value DNP 4.7k 1% OLED SDA pull-up to 3V3 -> DNP 4.7k 1% OLED SDA pull-up to AUX_3V3
- R11: value DNP 4.7k 1% OLED SCL pull-up to 3V3 -> DNP 4.7k 1% OLED SCL pull-up to AUX_3V3
Connections:
- net 5V_SYS: now also C10.2, C8.2, C9.1, C9.2, J6.1 (GND), J9.1 (5V_SYS), J9.3 (GND), JP1.1 (5V_SYS), R4.2, U4.1 (GND), U4.3 (IN); no longer J1.1 (VIN / 5V)
- net BAT_FUSED: now also J8.1 (BAT_FUSED); no longer Q1.3 (D)
- net BUCK_IN: now also R3.1
- net DEVKIT_3V3: no longer J5.2 (VCC / 3V3), R10.2, R11.2
- net BAT_SENSE: now reaches J1.10 (GPIO32)
- net BAT_SENSE: now also C8.1, R3.2, R4.1
- net GPIO13: now reaches J1.3 (GPIO13)
- net GPIO13: now also J6.2 (GPIO13)
- net GPIO14: now reaches J1.5 (GPIO14)
- net GPIO14: now also J6.3 (GPIO14)
- net GPIO19: now reaches J2.10 (GPIO19)
- net GPIO19: now also J6.5 (GPIO19)
- net GPIO23: now reaches J2.15 (GPIO23)
- net GPIO23: now also J6.6 (GPIO23)
- net GPIO18: now reaches J2.9 (GPIO18)
- net GPIO18: now also J6.4 (GPIO18)
- net WS2812_DIN renamed WS2812_DATA_5V
- net WS2812_DATA_5V: now also J9.2 (WS2812_DATA_5V)
- new net AUX_3V3: C10.1, J5.2 (VCC / 3V3), R10.2, R11.2, U4.2 (OUT / TAB)
- new net BAT_SW: J8.2 (BAT_SW), Q1.3 (D)
- new net DEVKIT_VIN: J1.1 (VIN / 5V), JP1.2 (DEVKIT_VIN)
- no-connect marks 20 -> 13
Other:
- note added: "5V_SYS ALLOCATION: 985.692mA WITH 20% MARGIN; J_RGB POLICY MAXIMUM 3 x WS2812B-V5 (109.800mA ALLOCATION)."
- note added: "A1. BATTERY SENSE (GPIO32 / ADC1_CH4)"
- note added: "AUX_3V3 ALLOCATION: OLED/J5 ONLY, 100mA. J6 HAS NO POWER PIN. DEVKIT_3V3 IS NOT FOR EXTERNAL ACCESSORIES."
- note added: "BAT+ -> F1 -> BAT_FUSED -> J8.1 -> EXTERNAL MECHANICAL SWITCH -> J8.2 -> BAT_SW -> Q1.3 -> BUCK_IN"
- note added: "BUCK_IN -> R3 10k 1% -> BAT_SENSE -> R4 3.3k 1% -> GND | C8 100nF BAT_SENSE-to-GND"
- note added: "ESP32 DEVKIT, E220, OLED, BUTTON PANEL AND RGB CHAIN ARE USER-INSTALLED."
- note added: "F. EXTERNAL WS2812 OUTPUT"
- note added: "G. BUTTON PANEL"
- note added: "GPIO4 -> U3 AHCT -> J_RGB.2 | J_RGB: 1 5V_SYS, 2 DATA, 3 GND | MAX 3 PIXELS"
- note added: "H. AUX_3V3 LDO"
- note added: "J5: 1 GND | 2 AUX_3V3 | 3 GPIO22/SCL | 4 GPIO21/SDA | R10/R11 4.7k DNP to AUX_3V3"
- note added: "J6 BUTTONS: 1 GND 2 GPIO13 3 GPIO14 4 GPIO18 5 GPIO19 6 GPIO23"
- note added: "J6 BUTTONS: ACTIVE-LOW CONTACTS TO GND ONLY; ENABLE FIRMWARE PULL-UPS; NO EXTERNAL VOLTAGE / NO GENERAL GPIO USE."
- note added: "J6: USER INSTALL / PCBA DNP; NORMALLY-OPEN ACTIVE-LOW CONTACTS TO GND ONLY; NOT A GENERAL-PURPOSE HEADER."
- note added: "JP1 DEVKIT_PWR: 5V_SYS -> JP1.1 -> removable shunt -> JP1.2 -> DEVKIT_VIN -> J1.1"
- note added: "NO DISPLAY-AUX HEADER, SIGNAL TEST POINTS, OR ONBOARD RGB PIXEL IN THIS REVISION."
- note added: "NORMAL: POWER_SW ON + JP1 CLOSED. USB SERVICE: POWER_SW OFF + JP1 OPEN WHEN ISOLATION IS DESIRED. GPIO IS NOT AUTOMATICALLY/COMPLETELY ISOLATED."
- note added: "U4 THERMAL POLICY @ 100.1mA 5V_SYS ALLOCATION: PAD1=GND; PAD2 LEAD+TAB=AUX_3V3; PAD3=5V_SYS. USE ORDINARY PROPORTIONATE LOCAL F.Cu ON OUT/TAB; B.Cu AUX_3V3 ISLAND / THERMAL-VIA ARRAY ONLY IF ANALYSIS REQUIRES."
- note added: "U4 TLV1117LV33DCYR: 5V_SYS -> 3.3V AUX_3V3 | C9/C10 10uF X5R close to U4 | DCY tab = OUT"
- note added: "USED: VIN via JP1, 3V3, GND | GPIO17/TX2, GPIO16/RX2, GPIO25/26/27, GPIO21/22, GPIO4, GPIO13/14/18/19/23/32"
- note removed: "BAT+ -> F1 -> BAT_FUSED -> Q1 -> BUCK_IN"
- note removed: "ESP32 DEVKIT, E220 AND OLED ARE USER-INSTALLED MODULES."
- note removed: "F. WS2812 STATUS LED"
- note removed: "GPIO4 -> AHCT buffer -> DIN"
- note removed: "J5: 1 GND | 2 DEVKIT_3V3 | 3 GPIO22/SCL | 4 GPIO21/SDA | R10/R11 4.7k DNP"
- note removed: "USED: VIN, 3V3, GND | GPIO17/TX2, GPIO16/RX2, GPIO25/26/27, GPIO21/22, GPIO4"

Commit message: Audit and correct production footprints
Parts:
- JP1: footprint Connector_PinHeader_2.54mm:PinHeader_1x02_P2.54mm_Vertical -> Carrier:Samtec_TSW-102-07-G-S_1x02_P2.54mm_THT
- U4: footprint Package_TO_SOT_SMD:SOT-223-3_TabPin2 -> Carrier:TI_TLV1117LV33DCYR_DCY_SOT223
Changed lines of the file:
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@@
       (effects (font (size 1.27 1.27)) hide)
     )
-    (property "Footprint" "Connector_PinHeader_2.54mm:PinHeader_1x02_P2.54mm_Vertical" (id 2) (at 85.09 69.85 0)
+    (property "Footprint" "Carrier:Samtec_TSW-102-07-G-S_1x02_P2.54mm_THT" (id 2) (at 85.09 69.85 0)
       (effects (font (size 1.27 1.27)) hide)
     )
@@
       (effects (font (size 1.27 1.27)) hide)
     )
-    (property "Footprint" "Package_TO_SOT_SMD:SOT-223-3_TabPin2" (id 2) (at 265.43 255.27 0)
+    (property "Footprint" "Carrier:TI_TLV1117LV33DCYR_DCY_SOT223" (id 2) (at 265.43 255.27 0)
       (effects (font (size 1.27 1.27)) hide)
     )
