File: hardware/evidence/project-state-reconciliation-2026-08-19/pre-metadata-title-text.kicad_pcb (KiCad board)
At the start: 2 copper layers, 145 x 90 mm, 33 parts, among them J1 SSW-115-02-G-S DEVKIT LEFT, J2 SSW-115-02-G-S DEVKIT RIGHT, J3 E220-400T22D / E220-900T22D S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, J4 B2B-XH-A, J5 SSW-104-02-G-S, Q1 DMP3130LQ-7, U1 TPS62133RGT, U3 SN74AHCT1G125DBVR

Commit message: next commit
Other:
- board text added: "STAGE 8 — FUNCTIONAL PLACEMENT ONLY / NO ROUTING"
- board text added: "U1 EP=GND. THERMAL VIAS / SW-COPPER POLICY: LAYOUT REVIEW REQUIRED"
- board text removed: "REV.1 CONTROLLED ROUTING — POWER + 5V PASSED / SIGNAL ROUTING PENDING"
- board text removed: "TPS62133 BUCK CELL — REVIEWED RETAINED CHECKPOINT"
Changed lines of the file:
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@@
 	(paper "A4")
 	(title_block
-		(title "ESP32 + E220 carrier — Rev.1 controlled routing")
-		(comment 1 "POWER + 5V ROUTING REVIEWED / SIGNAL ROUTING INCOMPLETE / NOT FOR PRODUCTION")
+		(title "ESP32 + E220 carrier — Stage 8 functional placement")
+		(comment 1 "UNROUTED / NOT FOR PRODUCTION")
 		(comment 2 "145 x 90 mm preferred comfortable preliminary outline")
 		(comment 3 "All active carrier components instantiated; R10/R11 DNP/no-footprint")
@@
 		)
 	)
-	(gr_text "TPS62133 BUCK CELL — REVIEWED RETAINED CHECKPOINT"
+	(gr_text "U1 EP=GND. THERMAL VIAS / SW-COPPER POLICY: LAYOUT REVIEW REQUIRED"
 		(at 62 88.2 0)
 		(layer "Dwgs.User")
@@
 		)
 	)
-	(gr_text "REV.1 CONTROLLED ROUTING — POWER + 5V PASSED / SIGNAL ROUTING PENDING"
+	(gr_text "STAGE 8 — FUNCTIONAL PLACEMENT ONLY / NO ROUTING"
 		(at 65 3.5 0)
 		(layer "Dwgs.User")
